Commit message: fix: bundle gripper meshes in repo for cross-machine portability
The combined URDF previously referenced gripper meshes via absolute
file:// paths into third_party/OnRobot-RG2FT-ROS/, which is gitignored.
On a fresh clone (e.g. lab PC), the meshes didn't exist and URDF import
failed.

Fix: copy the 18 STL files (9 visual + 9 collision, 7 MB total) into
isaac/gripper_meshes/ and update the URDF paths to reference
/workspace/isaac/gripper_meshes/ (bind-mounted in the container).

Now `git clone + container.sh start` provides everything needed —
no manual clone of OnRobot-RG2FT-ROS required.

Also updates generate_combined_urdf.sh to use the bundled mesh path,
and adds gripper_meshes/ to the README repo structure.

Co-Authored-By: Claude Opus 4.6 (1M context) <noreply@anthropic.com>

File: isaac/m1013_rg2ft_combined.urdf (robot description, URDF)
Before this commit: robot m1013, 16 links, 15 joints
Links:
- link angle_bracket: geometry collision mesh filename=file:///workspace/isaac/gripper_meshes/collision/angle_brac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 scale=0.001 0.001 0.001; visual mesh filename=file:///workspace/isaac/gripper_meshes/visual/angle_bracket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 scale=0.001 0.001 0.001
- link gripper_body: geometry collision mesh filename=file:///workspace/isaac/gripper_meshes/collision/gripper_bo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 scale=0.001 0.001 0.001; visual mesh filename=file:///workspace/isaac/gripper_meshes/visual/gripper_body.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 scale=0.001 0.001 0.001
- link left_inner_finger: geometry collision mesh filename=file:///workspace/isaac/gripper_meshes/collision/left_inner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 scale=0.001 0.001 0.001; visual mesh filename=file:///workspace/isaac/gripper_meshes/visual/left_inner_fi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 scale=0.001 0.001 0.001
- link left_inner_knuckle: geometry collision mesh filename=file:///workspace/isaac/gripper_meshes/collision/left_inner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 scale=0.001 0.001 0.001; visual mesh filename=file:///workspace/isaac/gripper_meshes/visual/left_inner_kn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 scale=0.001 0.001 0.001
- link left_outer_knuckle: geometry collision mesh filename=file:///workspace/isaac/gripper_meshes/collision/left_outer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 scale=0.001 0.001 0.001; visual mesh filename=file:///workspace/isaac/gripper_meshes/visual/left_outer_kn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 scale=0.001 0.001 0.001
- link quick_changer: geometry collision mesh filename=file:///workspace/isaac/gripper_meshes/collision/quick_chan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 scale=0.001 0.001 0.001; visual mesh filename=file:///workspace/isaac/gripper_meshes/visual/quick_changer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 scale=0.001 0.001 0.001
- link right_inner_finger: geometry collision mesh filename=file:///workspace/isaac/gripper_meshes/collision/right_inne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 scale=0.001 0.001 0.001; visual mesh filename=file:///workspace/isaac/gripper_meshes/visual/right_inner_f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 scale=0.001 0.001 0.001
- link right_inner_knuckle: geometry collision mesh filename=file:///workspace/isaac/gripper_meshes/collision/right_inne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 scale=0.001 0.001 0.001; visual mesh filename=file:///workspace/isaac/gripper_meshes/visual/right_inner_k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 scale=0.001 0.001 0.001
- link right_outer_knuckle: geometry collision mesh filename=file:///workspace/isaac/gripper_meshes/collision/right_oute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 scale=0.001 0.001 0.001; visual mesh filename=file:///workspace/isaac/gripper_meshes/visual/right_outer_k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 scale=0.001 0.001 0.001

Commit message: fix: rotate gripper mount 90° yaw to match real robot orientation
Co-Authored-By: Claude Opus 4.6 (1M context) <noreply@anthropic.com>

File: isaac/m1013_rg2ft_combined.urdf (robot description, URDF)
Before this commit: robot m1013, 16 links, 15 joints
Joints:
- joint quick_changer_joint: origin xyz=0 0 0 rpy=0 0 0 -> xyz=0 0 0 rpy=0 0 1.5708
